File: hardware/car.kicad_sch (KiCad schematic)
At the start: 23 parts, among them M1 Steering servo, SW1 E-Switch JS5208 five-way, U1 Seeed XIAO ESP32-S3 Sense, U2 Flywoo GOKU GM10 Nano (u-blox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, U3 Kyosho KR-331 receiver, U4 ESC with BEC (Brainz 8), U5 LSM6DSO32 IMU breakout, U6 5 V buck, 100 % duty, 5-8.4 V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, U7 74LVC2G17

Commit message: Power the car through an LM2940, clamp the RC inputs with BAT43s, keep the two keys
The car sheet's rev 2. An LM2940CT-5.0 in place of the 100 %-duty buck, and
no diodes in the power path: a servo plug cannot swap + and -, and the
regulator survives a reversed input on its own, so the USB is never plugged
in while the car or a LiPo powers the board (PLAN-ESP32.md §2.7). Each RC
input through 10 k, with a BAT43 clamp to 3V3 and 100 k to ground:
through-hole parts in place of the 74LVC2G17 (§2.5). The bench's two keys
go in the car too (§3.1).

The sheet is generated again from gen_schematics.py, as it had never been
edited in KiCad, with the UUIDs of what did not change kept; the ERC is
clean and every net was read. Three drawings in Italian show where each
wire goes: wiring-bench and wiring-car, written by gen_wiring.py, and the
power path pin by pin.

Co-Authored-By: Claude Opus 5.5 <noreply@anthropic.com>
Parts:
- removed C3: 100n, symbol Device:C
- removed R7: 100k, symbol Device:R
- removed SW1: E-Switch JS5208 five-way, symbol rct:JS5208
- removed U6: 5 V buck, 100 % duty, 5-8.4 V in, symbol rct:Buck_5V
- removed U7: 74LVC2G17, symbol 74xGxx:74LVC2G17
- added C3: 47u tantalum, symbol Device:C_Polarized
- added SW1: OK, symbol Switch:SW_Push
- added SW2: NAV, symbol Switch:SW_Push
- added U6: LM2940CT-5.0, symbol rct:LM2940CT-5.0
- C1: value 470u low ESR -> 470u
- D1, D2: value SS14 -> BAT43
- R2: value 2k2 -> 10k
- R3: value 4k7 -> 10k
- R5: value 22k -> 100k
Connections:
- net +3V3: now also D1.1 (K), D2.1 (K)
- net +5V: now also U1.14 (5V), C3.1, U6.3 (VO); no longer D2.2 (A)
- net CH1_STEER: now also R3.1; no longer R6.1
- net CH2_THROTTLE: now also R4.1
- net GND: now also R2.2, R5.2, C3.2, SW1.1, U6.2 (GND)
- net KEYS: now also SW1.2, SW2.2; no longer R2.2, R3.2, R4.2, R5.2
- net RC_STEER: now also D1.2 (A), R3.2, R5.1
- net RC_THROTTLE: now also D2.2 (A), R4.2, R6.1
- net RX_RAIL: now also C1.1, C2.1, U6.1 (VI); no longer D1.2 (A)
- net at R2.1: now also SW2.1
- removed net XIAO_5V: D2.1 (K), U1.14 (5V)
Other:
- note added: "Keys: the bench's two buttons (PLAN-ESP32.md 3.1): a 10 k pull-up on D0, OK straight to ground, NAV through 10 k; 0 V, 1.62 V, and 3.12 V at rest. The IMU shares the I2C bus with the display; the GM10 runs from the LM2940's 5 V."
- note added: "Power: never the receiver rail straight into the 5V pad. C1, low ESR, and C2 soak up the servo's spikes, and the LM2940 holds 5 V for the 5V pad and the GM10. It is guaranteed from 6.25 V in; on a 5.9 V BEC its dropout, 0.2 V at most at 100 mA, leaves room, to confirm on the bench. C3 keeps it stable: 22 u or more, ESR 0.1 to 1 ohm, so a tantalum or a low-ESR electrolytic, never a ceramic alone. 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"
- note added: "RC inputs, per channel: 10 k in series; a BAT43 to 3V3 that holds a 5 V receiver's pulse under the pin's 3.6 V; 100 k to ground that holds the pin low with the receiver off, as the RC inputs wake the chip. A 3.3 V receiver's high reads about 3.0 V, over the 2.48 V needed."
- note removed: "Keys: the JS5208's centre pulls D0 to ground; each direction does so through its resistor, against the 10 k pull-up: about 0.6, 1.05, 1.65 and 2.27 V (PLAN-ESP32.md 3.1). The IMU shares the I2C bus with the display; the GM10 runs from the buck's 5 V."
- note removed: "Power: never the receiver rail straight into the 5V pad. D1 guards against reverse polarity, C1 and C2 soak up the servo's spikes, and the buck holds 5 V from 5 to 8.4 V in. D2 keeps the car's 5 V and the USB's apart: to confirm against the XIAO's schematic, which may already isolate VBUS. The LiPo on the BAT pads carries the shutdown when the car is switched off."
- note removed: "RC front end: the buffer takes 3.3 V or 5 V logic and gives D2 and D3 a clean 3.3 V; the 100 k pull-downs hold its inputs low with the receiver off, as the RC inputs wake the chip."
- title: In the car: power, backup LiPo, buffered RC inputs, JS5208, IMU -> In the car: power, backup LiPo, protected RC inputs, two keys, IMU

Commit message: Stabilise the LM2940 with a low-ESR electrolytic, make the IMU optional
- C3, the LM2940's output capacitor, is a Panasonic EEU-FR1C101: 100 uF
  16 V at 0.3 ohm, inside the 0.1-1 ohm the regulator needs. The small
  dipped tantalums first drawn run 1.3-2 ohm, too high (PLAN-ESP32.md
  §2.7); C1 is its 470 uF sibling, EEU-FR1C471.
- The IMU is optional (§2.6): drawn crossed out in car.kicad_sch (DNP),
  dashed in wiring-car. It costs no pin, sharing the display's I2C bus at
  0x6A and read through its FIFO; mounting it rigid on the chassis is the
  harder part.
- wiring-power-ldo goes: wiring-car draws the LM2940's pins, and its
  checklist joins the car drawing's warnings.

Co-Authored-By: Claude Opus 5.5 <noreply@anthropic.com>
Parts:
- C3: value 47u tantalum -> 100u EEU-FR1C101
- U5: value LSM6DSO32 IMU breakout -> LSM6DSO32 IMU breakout, optional; now not fitted
Other:
- note added: "Keys: the bench's two buttons (PLAN-ESP32.md 3.1): a 10 k pull-up on D0, OK straight to ground, NAV through 10 k; 0 V, 1.62 V, and 3.12 V at rest. The IMU is optional (DNP): on the I2C bus with the display, at 0x6A, it needs no GPIO. The GM10 runs from the LM2940's 5 V."
- note added: "Power: never the receiver rail straight into the 5V pad. C1, low ESR, and C2 soak up the servo's spikes, and the LM2940 holds 5 V for the 5V pad and the GM10. It is guaranteed from 6.25 V in; on a 5.9 V BEC its dropout, 0.2 V at most at 100 mA, leaves room, to confirm on the bench. C3 keeps it stable: 22 u or more, ESR 0.1 to 1 ohm: a low-ESR electrolytic, the EEU-FR1C101, as small tantalums run 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"
- note removed: "Keys: the bench's two buttons (PLAN-ESP32.md 3.1): a 10 k pull-up on D0, OK straight to ground, NAV through 10 k; 0 V, 1.62 V, and 3.12 V at rest. The IMU shares the I2C bus with the display; the GM10 runs from the LM2940's 5 V."
- note removed: "Power: never the receiver rail straight into the 5V pad. C1, low ESR, and C2 soak up the servo's spikes, and the LM2940 holds 5 V for the 5V pad and the GM10. It is guaranteed from 6.25 V in; on a 5.9 V BEC its dropout, 0.2 V at most at 100 mA, leaves room, to confirm on the bench. C3 keeps it stable: 22 u or more, ESR 0.1 to 1 ohm, so a tantalum or a low-ESR electrolytic, never a ceramic alone. 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"
Changed lines of the file:
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@@
 	(wire (pts (xy 76.2 52.07) (xy 78.74 52.07)) (stroke (width 0) (type default)))
 	(label "SDA" (at 78.74 52.07 0) (effects (font (size 1.27 1.27)) (justify left bottom)))
-	(symbol (lib_id "rct:LSM6DSO32_breakout") (at 63.5 93.98 0) (unit 1) (exclude_from_sim no) (in_bom yes) (on_board yes) (dnp no) (property "Reference" "U5" (at 55.88 83.82 0) (effects (font (size 1.27 1.27)))) (property "Value" "LSM6DSO32 IMU breakout" (at 63.5 113.03 0) (effects (font (size 1.27 1.27)))) (property "Footprint" "" (at 63.5 93.98 0) (effects (font (size 1.27 1.27)) (hide yes))) (property "Datasheet" "~" (at 63.5 93.98 0) (effects (font (size 1.27 1.27)) (hide yes))) (pin "1") (pin "2") (pin "3") (pin "4") (instances (project "car" (path "/ffdedf3a-67e8-4282-b496-2684f4fc429c" (reference "U5") (unit 1)))))
+	(symbol (lib_id "rct:LSM6DSO32_breakout") (at 63.5 93.98 0) (unit 1) (exclude_from_sim no) (in_bom yes) (on_board yes) (dnp yes) (property "Reference" "U5" (at 55.88 83.82 0) (effects (font (size 1.27 1.27)))) (property "Value" "LSM6DSO32 IMU breakout, optional" (at 63.5 113.03 0) (effects (font (size 1.27 1.27)))) (property "Footprint" "" (at 63.5 93.98 0) (effects (font (size 1.27 1.27)) (hide yes))) (property "Datasheet" "~" (at 63.5 93.98 0) (effects (font (size 1.27 1.27)) (hide yes))) (pin "1") (pin "2") (pin "3") (pin "4") (instances (project "car" (path "/ffdedf3a-67e8-4282-b496-2684f4fc429c" (reference "U5") (unit 1)))))
 	(wire (pts (xy 63.5 82.55) (xy 63.5 80.01)) (stroke (width 0) (type default)))
 	(symbol (lib_id "power:+3V3") (at 63.5 80.01 0) (unit 1) (exclude_from_sim no) (in_bom yes) (on_board yes) (dnp no) (property "Reference" "#PWR006" (at 63.5 75.01 0) (effects (font (size 1.27 1.27)) (hide yes))) (property "Value" "+3V3" (at 63.5 76.2 0) (effects (font (size 1.27 1.27)))) (property "Footprint" "" (at 63.5 80.01 0) (effects (font (size 1.27 1.27)) (hide yes))) (property "Datasheet" "~" (at 63.5 80.01 0) (effects (font (size 1.27 1.27)) (hide yes))) (pin "1") (instances (project "car" (path "/ffdedf3a-67e8-4282-b496-2684f4fc429c" (reference "#PWR006") (unit 1)))))
@@
 	(wire (pts (xy 300.99 223.52) (xy 300.99 226.06)) (stroke (width 0) (type default)))
 	(symbol (lib_id "power:GND") (at 300.99 226.06 0) (unit 1) (exclude_from_sim no) (in_bom yes) (on_board yes) (dnp no) (property "Reference" "#PWR023" (at 300.99 221.06 0) (effects (font (size 1.27 1.27)) (hide yes))) (property "Value" "GND" (at 300.99 229.87 0) (effects (font (size 1.27 1.27)))) (property "Footprint" "" (at 300.99 226.06 0) (effects (font (size 1.27 1.27)) (hide yes))) (property "Datasheet" "~" (at 300.99 226.06 0) (effects (font (size 1.27 1.27)) (hide yes))) (pin "1") (instances (project "car" (path "/ffdedf3a-67e8-4282-b496-2684f4fc429c" (reference "#PWR023") (unit 1)))))
-	(symbol (lib_id "Device:C_Polarized") (at 313.69 222.25 0) (unit 1) (exclude_from_sim no) (in_bom yes) (on_board yes) (dnp no) (property "Reference" "C3" (at 318.77 220.98 0) (effects (font (size 1.27 1.27)))) (property "Value" "47u tantalum" (at 322.58 223.52 0) (effects (font (size 1.27 1.27)))) (property "Footprint" "" (at 313.69 222.25 0) (effects (font (size 1.27 1.27)) (hide yes))) (property "Datasheet" "~" (at 313.69 222.25 0) (effects (font (size 1.27 1.27)) (hide yes))) (pin "1") (pin "2") (instances (project "car" (path "/ffdedf3a-67e8-4282-b496-2684f4fc429c" (reference "C3") (unit 1)))))
+	(symbol (lib_id "Device:C_Polarized") (at 313.69 222.25 0) (unit 1) (exclude_from_sim no) (in_bom yes) (on_board yes) (dnp no) (property "Reference" "C3" (at 318.77 220.98 0) (effects (font (size 1.27 1.27)))) (property "Value" "100u EEU-FR1C101" (at 322.58 223.52 0) (effects (font (size 1.27 1.27)))) (property "Footprint" "" (at 313.69 222.25 0) (effects (font (size 1.27 1.27)) (hide yes))) (property "Datasheet" "~" (at 313.69 222.25 0) (effects (font (size 1.27 1.27)) (hide yes))) (pin "1") (pin "2") (instances (project "car" (path "/ffdedf3a-67e8-4282-b496-2684f4fc429c" (reference "C3") (unit 1)))))
 	(wire (pts (xy 313.69 215.9) (xy 313.69 218.44)) (stroke (width 0) (type default)))
 	(junction (at 313.69 215.9) (diameter 0) (color 0 0 0 0))
@@
 	(symbol (lib_id "power:GND") (at 25.4 27.94 0) (unit 1) (exclude_from_sim no) (in_bom yes) (on_board yes) (dnp no) (property "Reference" "#PWR027" (at 25.4 22.94 0) (effects (font (size 1.27 1.27)) (hide yes))) (property "Value" "GND" (at 25.4 31.75 0) (effects (font (size 1.27 1.27)))) (property "Footprint" "" (at 25.4 27.94 0) (effects (font (size 1.27 1.27)) (hide yes))) (property "Datasheet" "~" (at 25.4 27.94 0) (effects (font (size 1.27 1.27)) (hide yes))) (pin "1") (instances (project "car" (path "/ffdedf3a-67e8-4282-b496-2684f4fc429c" (reference "#PWR027") (unit 1)))))
 	(text "XIAO pads, USB-C up, from the top: left D0 D1 D2 D3 D4 D5 D6, right 5V GND 3V3 D10 D9 D8 D7;\nBAT+ and BAT- on the back. The microSD of the Sense board takes D8 CLK, D9 DAT0, D10 CMD and\nGPIO21 for DAT3, inside: leave D8-D10 free. D1 is spare, for the optional aux channel." (exclude_from_sim no) (at 20.32 193.04 0) (effects (font (size 1.27 1.27)) (justify left top)))
-	(text "Keys: the bench's two buttons (PLAN-ESP32.md 3.1): a 10 k pull-up on D0, OK straight to\nground, NAV through 10 k; 0 V, 1.62 V, and 3.12 V at rest.\nThe IMU shares the I2C bus with the display; the GM10 runs from the LM2940's 5 V." (exclude_from_sim no) (at 20.32 208.28 0) (effects (font (size 1.27 1.27)) (justify left top)))
+	(text "Keys: the bench's two buttons (PLAN-ESP32.md 3.1): a 10 k pull-up on D0, OK straight to\nground, NAV through 10 k; 0 V, 1.62 V, and 3.12 V at rest.\nThe IMU is optional (DNP): on the I2C bus with the display, at 0x6A, it needs no GPIO.\nThe GM10 runs from the LM2940's 5 V." (exclude_from_sim no) (at 20.32 208.28 0) (effects (font (size 1.27 1.27)) (justify left top)))
 	(text "RC inputs, per channel: 10 k in series; a BAT43 to 3V3 that holds a 5 V receiver's pulse\nunder the pin's 3.6 V; 100 k to ground that holds the pin low with the receiver off, as the\nRC inputs wake the chip. A 3.3 V receiver's high reads about 3.0 V, over the 2.48 V needed." (exclude_from_sim no) (at 236.22 190.5 0) (effects (font (size 1.27 1.27)) (justify left top)))
-	(text "Power: never the receiver rail straight into the 5V pad. C1, low ESR, and C2 soak up the\nservo's spikes, and the LM2940 holds 5 V for the 5V pad and the GM10. It is guaranteed from\n6.25 V in; on a 5.9 V BEC its dropout, 0.2 V at most at 100 mA, leaves room, to confirm on\nthe bench. C3 keeps it stable: 22 u or more, ESR 0.1 to 1 ohm, so a tantalum or a low-ESR\nelectrolytic, never a ceramic alone. No diodes (decided 2026-10-24), so the USB is never\nplugged in while the car or a LiPo powers the board: the two 5 V would meet on the 5V pad.\nThe LiPo on the BAT pads carries the shutdown when the car is switched off." (exclude_from_sim no) (at 20.32 226.06 0) (effects (font (size 1.27 1.27)) (justify left top)))
+	(text "Power: never the receiver rail straight into the 5V pad. C1, low ESR, and C2 soak up the\nservo's spikes, and the LM2940 holds 5 V for the 5V pad and the GM10. It is guaranteed from\n6.25 V in; on a 5.9 V BEC its dropout, 0.2 V at most at 100 mA, leaves room, to confirm on\nthe bench. C3 keeps it stable: 22 u or more, ESR 0.1 to 1 ohm: a low-ESR electrolytic, the\nEEU-FR1C101, as small tantalums run over 1 ohm. No diodes (decided 2026-10-24), so the\nUSB is never plugged in while the car or a LiPo powers the board: the two 5 V would meet\non the 5V pad.\nThe LiPo on the BAT pads carries the shutdown when the car is switched off." (exclude_from_sim no) (at 20.32 226.06 0) (effects (font (size 1.27 1.27)) (justify left top)))
 	(sheet_instances (path "/" (page "1"))) (embedded_fonts no))
