File: hardware/car.kicad_sch (KiCad schematic)
At the start: 22 parts, among them M1 Steering servo, SW1 OK, SW2 NAV, U1 Seeed XIAO ESP32-S3 Sense, U2 Flywoo GOKU GM10 Nano (u-blox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, U3 Kyosho KR-331 receiver, U4 ESC with BEC (Brainz 8), U5 LSM6DSO32 IMU breakout, optio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, U6 LM2940CT-5.0

Commit message: Close at boot a session the car's switch cut, and sleep from IDLE (ROADMAP 6.5)
There is no backup battery (decided 2026-10-25): the device goes off
with the car within a millisecond or so, so a session is ended by hand,
or by the automatic stop, before the switch. The 1S LiPo on BAT+/BAT-
leaves car.kicad_sch (rev 3; BT1 out, the pads unconnected, ERC clean,
only those nets changed) and the wiring drawing, and the status bar its
LiPo mark (PLAN-ESP32.md §2.7, §4.5).

A session the switch cuts is closed at the next boot: sessionBegin()
names it in NVS and sessionEnd() clears it, and sessionRecover() cuts
its .rcl after the last whole record and gives meta.json
`close: unclosed`, a line in /post.log. rcl::findTail() finds that
record reading the file in pieces, given up 64 KB past it, where the
extent holds whatever the card had (4 host tests). A file whose session
header is another session's is left alone.

The board sleeps from IDLE only (lib/ui/ui_power.h): the RC signal
stopping, or 5 min with no RC signal, no USB host and no key, give a
10 s notice that any key, the pulses or a host cancel. A session is
never ended by the pulses. src/power.cpp switches the display off,
unmounts the card and sleeps until OK; /post.log names the wake.

The sim build gains `reset`, a restart that closes nothing, and
`usb off`, and wakes on a 20 s timer too. On it: a session reset 8.5 s
in was closed at the next boot in 170 ms, 106 records and 8,052 of
4,194,304 bytes kept, read back with no byte skipped, meta.json
`close: unclosed`; the notice counted down, OK cancelled it, and left
alone it slept and woke into the POST. 210 host tests.

Co-Authored-By: Claude Opus 5.5 <noreply@anthropic.com>
Parts:
- removed BT1: 1S LiPo 150-300 mAh, symbol Device:Battery_Cell
Connections:
- no-connect marks 5 -> 7
Other:
- note added: "RC inputs, per channel: 10 k in series; a BAT43 to 3V3 that holds a 5 V receiver's pulse under the pin's 3.6 V; 100 k to ground that holds the pin low with its lead unplugged, so that noise is not taken for pulses. A 3.3 V receiver's high reads about 3.0 V, over 2.48 V."
- note removed: "RC inputs, per channel: 10 k in series; a BAT43 to 3V3 that holds a 5 V receiver's pulse under the pin's 3.6 V; 100 k to ground that holds the pin low with the receiver off, as the RC inputs wake the chip. A 3.3 V receiver's high reads about 3.0 V, over the 2.48 V needed."
- title: In the car: power, backup LiPo, protected RC inputs, two keys, IMU -> In the car: power, protected RC inputs, two keys, IMU
Changed lines of the file:
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@@
-(kicad_sch (version 20250114) (generator "eeschema") (generator_version "9.0") (paper "A3") (title_block (title "In the car: power, backup LiPo, protected RC inputs, two keys, IMU") (date "2026-10-24") (rev "2") (company "esp32-rc-telemetry") (comment 1 "Signals and keys as on bench.kicad_sch; the power and the RC inputs' protection change.") (comment 2 "To confirm on the bench: the LM2940 on a 5.9 V BEC, the RC inputs' clamps, the IMU.") (comment 3 "The design of PLAN-ESP32.md 2.5, 2.7 and 3.1: not built yet."))
+(kicad_sch (version 20250114) (generator "eeschema") (generator_version "9.0") (paper "A3") (title_block (title "In the car: power, protected RC inputs, two keys, IMU") (date "2026-10-25") (rev "3") (company "esp32-rc-telemetry") (comment 1 "Signals and keys as on bench.kicad_sch; the power and the RC inputs' protection change.") (comment 2 "To confirm on the bench: the LM2940 on a 5.9 V BEC, the RC inputs' clamps, the IMU.") (comment 3 "The design of PLAN-ESP32.md 2.5, 2.7 and 3.1: not built yet."))
 	(symbol (lib_id "rct:XIAO_ESP32S3_Sense") (at 200.66 101.6 0) (unit 1) (exclude_from_sim no) (in_bom yes) (on_board yes) (dnp no) (property "Reference" "U1" (at 182.88 85.09 0) (effects (font (size 1.27 1.27)))) (property "Value" "Seeed XIAO ESP32-S3 Sense" (at 200.66 129.54 0) (effects (font (size 1.27 1.27)))) (property "Footprint" "" (at 200.66 101.6 0) (effects (font (size 1.27 1.27)) (hide yes))) (property "Datasheet" "~" (at 200.66 101.6 0) (effects (font (size 1.27 1.27)) (hide yes))) (pin "1") (pin "10") (pin "11") (pin "12") (pin "13") (pin "14") (pin "15") (pin "16") (pin "2") (pin "3") (pin "4") (pin "5") (pin "6") (pin "7") (pin "8") (pin "9") (instances (project "car" (path "/ffdedf3a-67e8-4282-b496-2684f4fc429c" (reference "U1") (unit 1)))))
 	(wire (pts (xy 177.8 93.98) (xy 175.26 93.98)) (stroke (width 0) (type default)))
@@
 	(wire (pts (xy 190.5 119.38) (xy 190.5 121.92)) (stroke (width 0) (type default)))
 	(symbol (lib_id "power:GND") (at 190.5 121.92 0) (unit 1) (exclude_from_sim no) (in_bom yes) (on_board yes) (dnp no) (property "Reference" "#PWR003" (at 190.5 116.92 0) (effects (font (size 1.27 1.27)) (hide yes))) (property "Value" "GND" (at 190.5 125.73 0) (effects (font (size 1.27 1.27)))) (property "Footprint" "" (at 190.5 121.92 0) (effects (font (size 1.27 1.27)) (hide yes))) (property "Datasheet" "~" (at 190.5 121.92 0) (effects (font (size 1.27 1.27)) (hide yes))) (pin "1") (instances (project "car" (path "/ffdedf3a-67e8-4282-b496-2684f4fc429c" (reference "#PWR003") (unit 1)))))
-	(symbol (lib_id "Device:Battery_Cell") (at 223.52 129.54 0) (unit 1) (exclude_from_sim no) (in_bom yes) (on_board yes) (dnp no) (property "Reference" "BT1" (at 227.33 128.27 0) (effects (font (size 1.27 1.27)))) (property "Value" "1S LiPo 150-300 mAh" (at 227.33 130.81 0) (effects (font (size 1.27 1.27)))) (property "Footprint" "" (at 223.52 129.54 0) (effects (font (size 1.27 1.27)) (hide yes))) (property "Datasheet" "~" (at 223.52 129.54 0) (effects (font (size 1.27 1.27)) (hide yes))) (pin "1") (pin "2") (instances (project "car" (path "/ffdedf3a-67e8-4282-b496-2684f4fc429c" (reference "BT1") (unit 1)))))
-	(wire (pts (xy 210.82 119.38) (xy 210.82 124.46)) (stroke (width 0) (type default)))
-	(wire (pts (xy 210.82 124.46) (xy 223.52 124.46)) (stroke (width 0) (type default)))
-	(wire (pts (xy 200.66 119.38) (xy 200.66 134.62)) (stroke (width 0) (type default)))
-	(wire (pts (xy 200.66 134.62) (xy 223.52 134.62)) (stroke (width 0) (type default)))
-	(wire (pts (xy 223.52 134.62) (xy 223.52 132.08)) (stroke (width 0) (type default)))
+	(no_connect (at 210.82 119.38))
+	(no_connect (at 200.66 119.38))
 	(symbol (lib_id "rct:SSD1306_OLED") (at 63.5 50.8 0) (unit 1) (exclude_from_sim no) (in_bom yes) (on_board yes) (dnp no) (property "Reference" "DS1" (at 55.88 40.64 0) (effects (font (size 1.27 1.27)))) (property "Value" "OLED 0.96in SSD1306 0x3C" (at 63.5 69.85 0) (effects (font (size 1.27 1.27)))) (property "Footprint" "" (at 63.5 50.8 0) (effects (font (size 1.27 1.27)) (hide yes))) (property "Datasheet" "~" (at 63.5 50.8 0) (effects (font (size 1.27 1.27)) (hide yes))) (pin "1") (pin "2") (pin "3") (pin "4") (instances (project "car" (path "/ffdedf3a-67e8-4282-b496-2684f4fc429c" (reference "DS1") (unit 1)))))
 	(wire (pts (xy 63.5 39.37) (xy 63.5 36.83)) (stroke (width 0) (type default)))
@@
 	(text "XIAO pads, USB-C up, from the top: left D0 D1 D2 D3 D4 D5 D6, right 5V GND 3V3 D10 D9 D8 D7;\nBAT+ and BAT- on the back. The microSD of the Sense board takes D8 CLK, D9 DAT0, D10 CMD and\nGPIO21 for DAT3, inside: leave D8-D10 free. D1 is spare, for the optional aux channel." (exclude_from_sim no) (at 20.32 193.04 0) (effects (font (size 1.27 1.27)) (justify left top)))
 	(text "Keys: the bench's two buttons (PLAN-ESP32.md 3.1): a 10 k pull-up on D0, OK straight to\nground, NAV through 10 k; 0 V, 1.62 V, and 3.12 V at rest.\nThe IMU is optional (DNP): on the I2C bus with the display, at 0x6A, it needs no GPIO.\nThe GM10 runs from the LM2940's 5 V." (exclude_from_sim no) (at 20.32 208.28 0) (effects (font (size 1.27 1.27)) (justify left top)))
-	(text "RC inputs, per channel: 10 k in series; a BAT43 to 3V3 that holds a 5 V receiver's pulse\nunder the pin's 3.6 V; 100 k to ground that holds the pin low with the receiver off, as the\nRC inputs wake the chip. A 3.3 V receiver's high reads about 3.0 V, over the 2.48 V needed." (exclude_from_sim no) (at 236.22 190.5 0) (effects (font (size 1.27 1.27)) (justify left top)))
-	(text "Power: never the receiver rail straight into the 5V pad. C1, low ESR, and C2 soak up the\nservo's spikes, and the LM2940 holds 5 V for the 5V pad and the GM10. It is guaranteed from\n6.25 V in; on a 5.9 V BEC its dropout, 0.2 V at most at 100 mA, leaves room, to confirm on\nthe bench. C3 keeps it stable: 22 u or more, ESR 0.1 to 1 ohm: a low-ESR electrolytic, the\nEEU-FR1C101, as small tantalums run over 1 ohm. No diodes (decided 2026-10-24), so the\nUSB is never plugged in while the car or a LiPo powers the board: the two 5 V would meet\non the 5V pad.\nThe LiPo on the BAT pads carries the shutdown when the car is switched off." (exclude_from_sim no) (at 20.32 226.06 0) (effects (font (size 1.27 1.27)) (justify left top)))
+	(text "RC inputs, per channel: 10 k in series; a BAT43 to 3V3 that holds a 5 V receiver's pulse\nunder the pin's 3.6 V; 100 k to ground that holds the pin low with its lead unplugged, so\nthat noise is not taken for pulses. A 3.3 V receiver's high reads about 3.0 V, over 2.48 V." (exclude_from_sim no) (at 236.22 190.5 0) (effects (font (size 1.27 1.27)) (justify left top)))
+	(text "Power: never the receiver rail straight into the 5V pad. C1, low ESR, and C2 soak up the\nservo's spikes, and the LM2940 holds 5 V for the 5V pad and the GM10. It is guaranteed from\n6.25 V in; on a 5.9 V BEC its dropout, 0.2 V at most at 100 mA, leaves room, to confirm on\nthe bench. C3 keeps it stable: 22 u or more, ESR 0.1 to 1 ohm: a low-ESR electrolytic, the\nEEU-FR1C101, as small tantalums run over 1 ohm. No diodes (decided 2026-10-24), so the\nUSB is never plugged in while the car or a LiPo powers the board: the two 5 V would meet\non the 5V pad.\nNo backup battery on BAT+/BAT- (decided 2026-10-25): the device goes off with the car, so\na session is ended by hand first; one the switch cuts is closed at the next boot." (exclude_from_sim no) (at 20.32 226.06 0) (effects (font (size 1.27 1.27)) (justify left top)))
 	(sheet_instances (path "/" (page "1"))) (embedded_fonts no))
